File: PCB/banc_rodage_pcb/banc_rodage_pcb.kicad_sch (KiCad schematic)
At the start: 37 parts, among them J1 CONN_HALL, J10 CONN_THERMISTANCE_MOSFET_3, J11 CONN_THERMISTANCE_MOSFET_4, J12 CONN_NEXTION, J13 Conn_01x14_Pin, J14 CONN_THERMISTANCE_MOTEUR, J2 CONN_MOTEUR, J3 CONN_ALIM, J4 CONN_CHAUFFE, J5 CONN_VENTIL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

Commit message: cleanup. automode : gestion of brenkin profile with the sd card (rename, duplicate, delete) is ok
Parts:
- removed C1: 0.33uf, Capacitor_THT:C_Rect_L4.0mm_W2.5mm_P2.50mm, symbol Device:C
- removed C2: 0.1uf, Capacitor_THT:C_Rect_L4.0mm_W2.5mm_P2.50mm, symbol Device:C
- removed J13: Conn_01x14_Pin, Connector_PinHeader_2.54mm:PinHeader_1x14_P2.54mm_Vertical, symbol Connector:Conn_01x16_Pin
- removed U3: LM78M05_TO252, Package_TO_SOT_THT:TO-220-3_Vertical, symbol Regulator_Linear:LM78M05_TO252
- added A1: Arduino_Nano_R4, arduino nano r4:Arduino_Nano_R4, symbol arduino nano R4:Arduino_Nano_R4
- added J15: CONN_ALIM_5, perso:TerminalBlock_bornier-2_P5.08mm, symbol Connector:Conn_01x02_Pin
- added U1: CAT24C256, Package_DIP:DIP-8_W7.62mm_Socket, symbol Memory_EEPROM:CAT24C256
- J10: value CONN_THERMISTANCE_MOSFET_3 -> NTC_MOSFET_3
- J11: value CONN_THERMISTANCE_MOSFET_4 -> NTC_MOSFET_4
- J14: value CONN_THERMISTANCE_MOTEUR -> NTC_MOTOR
- J2, J4, J7: footprint Perso:TerminalBlock_bornier-2_P5.08mm -> perso:TerminalBlock_bornier-2_P5.08mm
- J3: value CONN_ALIM -> CONN_ALIM_24; footprint Perso:TerminalBlock_bornier-2_P5.08mm -> perso:TerminalBlock_bornier-2_P5.08mm
- J6: value CONN_THERMISTANCE -> NTC_OIL
- J8: value CONN_THERMISTANCE_MOSFET_1 -> NTC_MOSFET_1
- J9: value CONN_THERMISTANCE_MOSFET_2 -> NTC_MOSFET_2
- Q1, Q2, Q3, Q4: footprint Perso:TO-220F-3_Horizontal_TabUp -> perso:TO-220F-3_Horizontal_TabUp
- R1, R10, R11, R2, R3, R4, R5, R6, R7, R8, R9: footprint Resistor_THT:R_Axial_DIN0207_L6.3mm_D2.5mm_P7.62mm_Horizontal -> Resistor_SMD:R_1206_3216Metric
Connections:
- net 3v3 is gone; now on net +5V: J1.1 (Pin_1), J10.1 (Pin_1), J11.1 (Pin_1), J14.1 (Pin_1), J6.1 (Pin_1), J8.1 (Pin_1), J9.1 (Pin_1)
- net +5V: now also A1.5V, J15.1 (Pin_1), U1.8 (VCC)
- net BUZZER+: now also A1.D4 (D4_CAN0_TX)
- net GND: now also J12.4 (Pin_4), A1.GND1 (GND), A1.GND2 (GND), J15.2 (Pin_2), U1.1 (A0), U1.2 (A1), U1.3 (A2), U1.4 (GND), U1.7 (WP); no longer J12.2 (Pin_2)
- net NEXTION_RX: now also A1.D1 (D1/TX)
- net NEXTION_TX: now also J12.2 (Pin_2), A1.D0 (D0/RX); no longer J12.4 (Pin_4)
- net SIGN_HALL: now also A1.D3 (D3_INT1)
- net ARDUINO_SIGN_CHAUFFE renamed PIN_HEATER
- net PIN_HEATER: now also A1.D11 (D11_MOSI)
- net ARDUINO_SIGN_MOTEUR renamed PIN_MOTOR
- net PIN_MOTOR: now also A1.D10 (D10_SS)
- net CHAUFFE_1 renamed HEATER_1
- net CHAUFFE_2 renamed HEATER_2
- net MOTEUR renamed MOTOR
- net SIGN_CHAUFFE renamed SIGN_HEATER
- net SIGN_MOTEUR renamed SIGN_MOTOR
- net SIGN_TEMP_HUILE renamed PIN_NTC_OIL
- net PIN_NTC_OIL: now also A1.A6
- net SIGN_THERMISTANCE_MOSFET_1 renamed PIN_NTC_MOSFET_1
- net PIN_NTC_MOSFET_1: now also A1.A0 (A0_DAC)
- net SIGN_THERMISTANCE_MOSFET_2 renamed PIN_NTC_MOSFET_2
- net PIN_NTC_MOSFET_2: now also A1.A1
- net SIGN_THERMISTANCE_MOSFET_3 renamed PIN_NTC_MOSFET_3
- net PIN_NTC_MOSFET_3: now also A1.A2
- net SIGN_THERMISTANCE_MOSFET_4 renamed PIN_NTC_MOSFET_4
- net PIN_NTC_MOSFET_4: now also A1.A3
- net SIGN_THERMISTANCE_MOTEUR renamed PIN_NTC_MOTOR
- net PIN_NTC_MOTOR: now also A1.A7
- new net: A1.A4 (A4/SDA), U1.5 (SDA)
- new net: A1.A5 (A5/SCL), U1.6 (SCL)
- no-connect marks 1 -> 16
Other:
- note added: "v1 : premiere edition v1.1 : ajout diode roue libre, ajout buzzer et pin. Nano R4."
- note removed: "v1 : premiere edition v1.1 : ajout diode roue libre, ajout buzzer et pin"
- moved on the sheet: BZ1, D1, D2, J1, J12, J2, J3, J4, J6, J7, Q1, Q2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
